Commit message: pick & place with mobile base manipulator

File: src/irb120_ros2_gazebo/urdf/irb120_macro.urdf.xacro (robot description, xacro)
@@ -445,4 +445,9 @@
         </geometry>
       </visual>
+      <collision>
+        <geometry>
+          <box size="0.001 0.001 0.001" />
+        </geometry>
+      </collision>
     </link>
     <joint name="EE_egp64_joint" type="prismatic">
