Commit message: increase weight of base robot and shift lidar to appropriate place

File: src/mobile_manipulator_body/urdf/robot_base.urdf.xacro (robot description, xacro)
@@ -13,12 +13,12 @@
     <inertial>
       <origin xyz="0.0030946 4.78250032638821E-11 0.053305" rpy="0 0 0" />
-      <mass value="47.873" />
-      <inertia
-        ixx="0.774276574699151"
-        ixy="-1.03781944357671E-10"
-        ixz="0.00763014265820928"
-        iyy="1.64933255189991"
-        iyz="1.09578155845563E-12"
-        izz="2.1239326987473" />
+      <mass value="500" />
+      <inertia
+        ixx="7.74276574699151"
+        ixy="-10.3781944357671E-10"
+        ixz="0.0763014265820928"
+        iyy="16.4933255189991"
+        iyz="10.9578155845563E-12"
+        izz="21.239326987473" />
     </inertial>
     <visual>
@@ -186,5 +186,5 @@
     <parent link="base_link" />
     <child link="base_scan" />
-    <origin xyz="-0.032 0 0.172" rpy="0 0 0" />
+    <origin xyz="0.2 0 0.172" rpy="0 0 0" />
   </joint>
   <gazebo reference="base_scan">

Commit message: Integrate moveit2 on abb robot with mobile base

File: src/mobile_manipulator_body/urdf/robot_base.urdf.xacro (robot description, xacro)
@@ -1,7 +1,13 @@
 <?xml version="1.0"?>
 <robot name="robot_base" xmlns:xacro="http://www.ros.org/wiki/xacro">
+  <!-- <link name="world" /> -->
   <!-- BASE LINK -->
   <link name="base_link">
   </link>
+  <!-- <joint name="world_to_base_link" type="fixed">
+    <parent link="world" />
+    <child link="base_link" />
+    <origin xyz="0.0 0.0 0.0" rpy="0.0 0.0 0.0" />
+  </joint> -->
   <!-- BASE_FOOTPRINT LINK -->
   <joint name="base_footprint_joint" type="fixed">

Commit message: add office world, mapping inside the room and navigation, add camera to the urdf and simulation environment

File: src/mobile_manipulator_body/urdf/robot_base.urdf.xacro (robot description, xacro)
@@ -205,5 +205,5 @@
         <range>
           <min>0.12</min>
-          <max>3.5</max>
+          <max>6</max>
         </range>
         <noise>
@@ -223,4 +223,51 @@
     </sensor>
   </gazebo>
+<!--  -->
+  <joint name="camera_joint" type="fixed">
+    <parent link="base_link"/>
+    <child link="camera_link"/>
+    <origin xyz="0.325 0 0.15" rpy="0 0 0"/>
+  </joint>
+  <link name="camera_link">
+      <visual>
+      <origin xyz="0 0 0.0" rpy="0 1.57 0" />
+      <geometry>
+        <mesh filename="file://$(find mobile_manipulator_body)/meshes/cam.stl"
+          scale="0.001 0.001 0.001" />
+      </geometry>
+      <!-- <material name="dark" /> -->
+      <color rgba="1 1 1 1" />
+    </visual>
+  </link>
+  <joint name="camera_optical_joint" type="fixed">
+    <parent link="camera_link"/>
+    <child link="camera_link_optical"/>
+    <origin xyz="0 0 0" rpy="${-pi/2} 0 ${-pi/2}"/>
+  </joint>
+  <link name="camera_link_optical"></link>
+   <gazebo reference="camera_link">
+      <material>Gazebo/Red</material>
+      <sensor name="camera" type="camera">
+        <pose> 0 0 0 0 0 0 </pose>
+        <visualize>true</visualize>
+        <update_rate>10</update_rate>
+        <camera>
+          <horizontal_fov>1.089</horizontal_fov>
+          <image>
+            <format>R8G8B8</format>
+            <width>640</width>
+            <height>480</height>
+          </image>
+          <clip>
+            <near>0.05</near>
+            <far>8.0</far>
+          </clip>
+        </camera>
+        <plugin name="camera_controller" filename="libgazebo_ros_camera.so">
+            <frame_name>camera_link_optical</frame_name>
+        </plugin>
+      </sensor>
+   </gazebo>
+            <!--  -->
   <joint name="front_left_wheel_joint" type="continuous">
     <axis xyz="0 1 0" />

Commit message: add navigation to ros2_execution, new map to hello.world, add camera

File: src/mobile_manipulator_body/urdf/robot_base.urdf.xacro (robot description, xacro)
@@ -204,12 +204,12 @@
         <scan>
           <horizontal>
-            <samples>360</samples>
-            <min_angle>0.00</min_angle>
-            <max_angle>6.28000</max_angle>
+            <samples>270</samples>
+            <min_angle>-2.356</min_angle>
+            <max_angle>2.356</max_angle>
           </horizontal>
         </scan>
         <range>
           <min>0.12</min>
-          <max>3.5</max>
+          <max>6</max>
         </range>
         <noise>
@@ -229,4 +229,60 @@
     </sensor>
   </gazebo>
+  <!--  -->
+  <joint name="camera_joint" type="fixed">
+    <parent link="base_link"/>
+    <child link="camera_link"/>
+    <origin xyz="0.325 0 0.15" rpy="0 0 0"/>
+  </joint>
+  <link name="camera_link">
+      <visual>
+      <origin xyz="0 0 0.0" rpy="0 1.57 0" />
+      <geometry>
+        <mesh filename="file://$(find mobile_manipulator_body)/meshes/cam.stl"
+          scale="0.001 0.001 0.001" />
+      </geometry>
+      <!-- <material name="dark" /> -->
+      <material name= "">
+        <color rgba="1 1 1 1" />
+      </material>
+    </visual>
+    <collision>
+      <origin xyz="0 0 0.0" rpy="0 1.57 0" />
+      <geometry>
+        <mesh filename="file://$(find mobile_manipulator_body)/meshes/cam.stl"
+          scale="0.001 0.001 0.001" />
+      </geometry>
+    </collision>
+  </link>
+  <joint name="camera_optical_joint" type="fixed">
+    <parent link="camera_link"/>
+    <child link="camera_link_optical"/>
+    <origin xyz="0 0 0" rpy="${-pi/2} 0 ${-pi/2}"/>
+  </joint>
+  <link name="camera_link_optical"></link>
+  <gazebo reference="camera_link">
+    <material>Gazebo/Red</material>
+    <sensor name="camera" type="camera">
+      <pose> 0 0 0 0 0 0 </pose>
+      <visualize>true</visualize>
+      <update_rate>10</update_rate>
+      <camera>
+        <horizontal_fov>1.089</horizontal_fov>
+        <image>
+          <format>R8G8B8</format>
+          <width>640</width>
+          <height>480</height>
+        </image>
+        <clip>
+          <near>0.05</near>
+          <far>8.0</far>
+        </clip>
+      </camera>
+      <plugin name="camera_controller" filename="libgazebo_ros_camera.so">
+          <frame_name>camera_link_optical</frame_name>
+      </plugin>
+    </sensor>
+  </gazebo>
+            <!--  -->
   <joint name="front_left_wheel_joint" type="continuous">
     <axis xyz="0 1 0" />
@@ -287,29 +343,29 @@
   </gazebo>
   <gazebo reference="front_left_wheel">
-    <mu1 value="1.0" />
-    <mu2 value="1.0" />
-    <kp value="10000000.0" />
-    <kd value="1.0" />
+    <mu1 value="0.8" />
+    <mu2 value="0.8" />
+    <kp value="100000.0" />
+    <kd value="10.0" />
     <fdir1 value="1 0 0" />
   </gazebo>
   <gazebo reference="front_right_wheel">
-    <mu1 value="1.0" />
-    <mu2 value="1.0" />
-    <kp value="10000000.0" />
-    <kd value="1.0" />
+    <mu1 value="0.8" />
+    <mu2 value="0.8" />
+    <kp value="100000.0" />
+    <kd value="10.0" />
     <fdir1 value="1 0 0" />
   </gazebo>
   <gazebo reference="rear_left_wheel">
-    <mu1 value="1.0" />
-    <mu2 value="1.0" />
-    <kp value="10000000.0" />
-    <kd value="1.0" />
+    <mu1 value="0.8" />
+    <mu2 value="0.8" />
+    <kp value="100000.0" />
+    <kd value="10.0" />
     <fdir1 value="1 0 0" />
   </gazebo>
-  <gazebo reference="rear_left_wheel">
-    <mu1 value="1.0" />
-    <mu2 value="1.0" />
-    <kp value="10000000.0" />
-    <kd value="1.0" />
+  <gazebo reference="rear_right_wheel">
+    <mu1 value="0.8" />
+    <mu2 value="0.8" />
+    <kp value="100000.0" />
+    <kd value="10.0" />
     <fdir1 value="1 0 0" />
   </gazebo>

Commit message: added error bound in navigation in ros2_execution, tried to transform map to base_link frame: failed

File: src/mobile_manipulator_body/urdf/robot_base.urdf.xacro (robot description, xacro)
@@ -19,5 +19,5 @@
     <inertial>
       <origin xyz="0.0030946 4.78250032638821E-11 0.053305" rpy="0 0 0" />
-      <mass value="500" />
+      <mass value="100" />
       <inertia
         ixx="7.74276574699151"
@@ -161,4 +161,40 @@
     </collision>
   </link>
+<!-- CASTER WHEEL LINK -->
+    <!-- <joint name="caster_wheel_joint" type="fixed">
+        <parent link="base_link"/>
+        <child link="caster_wheel"/>
+        <origin xyz="0.24 0 0"/>
+    </joint>
+    <link name="caster_wheel">
+        <visual>
+            <geometry>
+                <sphere radius="0.1"/>
+            </geometry>
+            <material name="black"/>
+        </visual>
+        <collision>
+            <geometry>
+                <sphere radius="0.1"/>
+            </geometry>
+        </collision>
+       <inertial>
+        <origin xyz="-4.1867E-18 0.0068085 -1.65658661799998E-18" rpy="0 0 0" />
+        <mass
+          value="1.0" />
+        <inertia
+          ixx="0.05"
+          ixy="0.05"
+          ixz="0.05"
+          iyy="0.05"
+          iyz="0.-19"
+          izz="0.00856502765719703" />
+        </inertial>
+    </link>
+    <gazebo reference="caster_wheel">
+        <material>Gazebo/Black</material>
+        <mu1 value="0.001"/>
+        <mu2 value="0.001"/>
+    </gazebo> -->
   <link name="imu_link" />
   <joint name="imu_joint" type="fixed">
@@ -199,5 +235,5 @@
       <pose> 0 0 0 0 0 0 </pose>
       <always_on>true</always_on>
-      <visualize>true</visualize>
+      <visualize>false</visualize>
       <update_rate>5</update_rate>
       <ray>
@@ -265,5 +301,5 @@
     <sensor name="camera" type="camera">
       <pose> 0 0 0 0 0 0 </pose>
-      <visualize>true</visualize>
+      <visualize>false</visualize>
       <update_rate>10</update_rate>
       <camera>
@@ -285,5 +321,5 @@
   </gazebo>
             <!--  -->
-  <joint name="front_left_wheel_joint" type="continuous">
+  <joint name="front_left_wheel_joint" type="fixed">
     <axis xyz="0 1 0" />
     <parent link="base_link" />
@@ -291,5 +327,5 @@
     <origin rpy="0 0 0" xyz="0.220 0.250 0" />
   </joint>
-  <joint name="front_right_wheel_joint" type="continuous">
+  <joint name="front_right_wheel_joint" type="fixed">
     <axis xyz="0 1 0" />
     <parent link="base_link" />
@@ -317,5 +353,5 @@
       <wheel_diameter>0.2</wheel_diameter>
       <!-- Limits -->
-      <max_wheel_torque>200</max_wheel_torque>
+      <max_wheel_torque>500</max_wheel_torque>
       <max_wheel_acceleration>10.0</max_wheel_acceleration>
       <!-- Output -->
@@ -327,5 +363,5 @@
     </plugin>
   </gazebo>
-  <gazebo>
+  <!-- <gazebo>
     <plugin name="front_wheel" filename="libgazebo_ros_diff_drive.so">
       <left_joint>front_left_wheel_joint</left_joint>
@@ -341,34 +377,36 @@
       <publish_wheel_tf>true</publish_wheel_tf>
     </plugin>
-  </gazebo>
-  <gazebo reference="front_left_wheel">
-    <mu1 value="0.8" />
-    <mu2 value="0.8" />
-    <kp value="100000.0" />
-    <kd value="10.0" />
+  </gazebo> -->
+  <!-- Fixed Front Wheels -->
+<gazebo reference="front_left_wheel">
+    <mu1 value="0.0001" />
+    <mu2 value="0.0001" />
+    <!-- <kp value="500000.0" />
+    <kd value="50.0" />
+    <fdir1 value="0 0 0" /> -->
+</gazebo>
+<gazebo reference="front_right_wheel">
+    <mu1 value="0.0001" />
+    <mu2 value="0.0001" />
+    <!-- <kp value="500000.0" />
+    <kd value="50.0" />
+    <fdir1 value="0 0 0" /> -->
+</gazebo>
+<!-- Powered Rear Wheels -->
+<gazebo reference="rear_left_wheel">
+    <mu1 value="0.6" />
+    <mu2 value="0.6" />
+    <kp value="1000000.0" />
+    <kd value="100.0" />
     <fdir1 value="1 0 0" />
-  </gazebo>
-  <gazebo reference="front_right_wheel">
-    <mu1 value="0.8" />
-    <mu2 value="0.8" />
-    <kp value="100000.0" />
-    <kd value="10.0" />
+</gazebo>
+<gazebo reference="rear_right_wheel">
+    <mu1 value="0.6" />
+    <mu2 value="0.6" />
+    <kp value="1000000.0" />
+    <kd value="100.0" />
     <fdir1 value="1 0 0" />
-  </gazebo>
-  <gazebo reference="rear_left_wheel">
-    <mu1 value="0.8" />
-    <mu2 value="0.8" />
-    <kp value="100000.0" />
-    <kd value="10.0" />
-    <fdir1 value="1 0 0" />
-  </gazebo>
-  <gazebo reference="rear_right_wheel">
-    <mu1 value="0.8" />
-    <mu2 value="0.8" />
-    <kp value="100000.0" />
-    <kd value="10.0" />
-    <fdir1 value="1 0 0" />
-  </gazebo>
-  <transmission
+</gazebo>
+  <!-- <transmission
     name="front_left_wheel_trans" type="SimpleTransmission">
     <type>transmission_interface/SimpleTransmission</type>
@@ -391,5 +429,5 @@
       <hardwareInterface>hardware_interface/VelocityJointInterface</hardwareInterface>
     </joint>
-  </transmission>
+  </transmission> -->
   <transmission
     name="rear_left_wheel_trans" type="SimpleTransmission">
